File: hardware-kicad/seedsigner-luckfox-pico-mini-v2/seedsigner-luckfox-pico-mini.kicad_pcb (KiCad board)
At the start: 4 copper layers, 65 x 30 mm, 8 parts, among them U1 LuckFox_Pico_MINI, U2 WAVESHARELCD_PLUS_UART_PLUS_I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

Commit message: update pcbs
Parts:
- moved U1 1.20 mm to (10.7, 49.3)
Routing:
- net /SPI_SCLK: track 16.0 -> 34.8 mm
- net /KEY3: track 21.7 -> 24.3 mm
- net /I2C-SDA: track 54.6 -> 52.1 mm, vias 0 -> 1
- net /SPI_MOSI: track 22.6 -> 20.8 mm
- net GND: track 31.3 -> 32.9 mm, vias 79 -> 84
- net /I2C-SCL: track 50.8 -> 49.1 mm, vias 0 -> 1
- net /DC: track 10.1 -> 8.73 mm
- net /KEY2: track 87.7 -> 86.7 mm
- net /RST: track 34.7 -> 35.7 mm
- net /KEY1: track 84.5 -> 83.6 mm
- net /JOYSTICK_LEFT: track 31.8 -> 31.1 mm
- net /JOYSTICK_UP: track 43.3 -> 42.6 mm
- net +3.3V: track 89.7 -> 90.3 mm
- net /JOYSTICK_PRESS: track 46.8 -> 46.3 mm
Other:
- outline, holes or cut-outs redrawn
- board text added: "Luckfox Pico Mini - Zero Adaptor Stephen Rothery + Lightningspore v1.0.2"
- board text removed: "Luckfox Pico Mini - Zero Adaptor Stephen Rothery + Lightningspore v1.0.1"
